Commit message: change mu coeff

File: models/objects/black_cube.urdf (robot description, URDF)
Before this commit: robot black_cube, 1 links, 0 joints
Links:
- link black_cube: geometry collision box size=0.055 0.055 0.055; visual box size=0.055 0.055 0.055

File: models/objects/blue_cube.urdf (robot description, URDF)
Before this commit: robot blue_cube, 1 links, 0 joints
Links:
- link blue_cube: geometry collision box size=0.055 0.055 0.055; visual box size=0.055 0.055 0.055

File: models/objects/green_cube.urdf (robot description, URDF)
Before this commit: robot green_cube, 1 links, 0 joints
Links:
- link green_cube: geometry collision box size=0.055 0.055 0.055; visual box size=0.055 0.055 0.055

File: models/objects/red_cube.urdf (robot description, URDF)
Before this commit: robot red_cube, 1 links, 0 joints
Links:
- link red_cube: geometry collision box size=0.055 0.055 0.055; visual box size=0.055 0.055 0.055
